Commit message: [Sw] fixxing blank mesh issue

File: shimizu_gantry_system/urdf/shimizu_gantry_system.urdf (robot description, URDF)
Before this commit: robot shimizu_gantry_system, 9 links, 8 joints
Links:
- removed link link_1
- removed link link_2
- removed link link_3
- removed link link_4
- removed link link_5
- removed link link_6
- added link link1, mass 39.488; collision mesh filename=package://shimizu_gantry_system/meshes/link1.STL; visual mesh filename=package://shimizu_gantry_system/meshes/link1.STL
- added link link2, mass 26.224; collision mesh filename=package://shimizu_gantry_system/meshes/link2.STL; visual mesh filename=package://shimizu_gantry_system/meshes/link2.STL
- added link link3, mass 41.069; collision mesh filename=package://shimizu_gantry_system/meshes/link3.STL; visual mesh filename=package://shimizu_gantry_system/meshes/link3.STL
- added link link4, mass 2.0071; collision mesh filename=package://shimizu_gantry_system/meshes/link4.STL; visual mesh filename=package://shimizu_gantry_system/meshes/link4.STL
- added link link5, mass 3.6409; collision mesh filename=package://shimizu_gantry_system/meshes/link5.STL; visual mesh filename=package://shimizu_gantry_system/meshes/link5.STL
- added link link6, mass 0.22702; collision mesh filename=package://shimizu_gantry_system/meshes/link6.STL; visual mesh filename=package://shimizu_gantry_system/meshes/link6.STL
Joints:
- removed joint joint_1
- removed joint joint_2
- removed joint joint_3
- removed joint joint_4
- removed joint joint_5
- removed joint joint_6
- removed joint linear_joint_x_to_y
- removed joint linear_joint_y_to_base
- added joint joint1: type continuous, parent base, child link1, origin xyz=0.44563 5.7729 17.038 rpy=1.5708 0 0, axis 0 0 1
- added joint joint2: type continuous, parent link1, child link2, origin xyz=0.32 0.078 -0.1973 rpy=0 1.5708 0, axis 0 1 0
- added joint joint3: type continuous, parent link2, child link3, origin xyz=0 0 0.87 rpy=0 0 0, axis 0 1 0
- added joint joint4: type continuous, parent link3, child link4, origin xyz=0.83 -0.0665 0.225 rpy=0 0 0, axis 1 0 0
- added joint joint5: type continuous, parent link4, child link5, origin xyz=0.1995 0 0 rpy=0 0 0, axis 0 1 0
- added joint joint6: type continuous, parent link5, child link6, origin xyz=0.1665 -0.009 0 rpy=1.5708 0 -1.5708, axis 0 0 1
- added joint x_to_y: type prismatic, parent gantry_x, child gantry_y, origin xyz=8.5487 -16.257 7.5966 rpy=1.5708 0 1.5708, axis 1 0 0, limit lower=0 upper=0 effort=0 velocity=0
- added joint y_to_base: type prismatic, parent gantry_y, child base, origin xyz=16.87 -7.5966 2.4892 rpy=0 -1.5708 0, axis 1 0 0, limit lower=0 upper=0 effort=0 velocity=0

Commit message: [Hw] adding shimizu_gantry_system

File: shimizu_gantry_system/urdf/shimizu_gantry_system.urdf (robot description, URDF)
Before this commit: robot shimizu_gantry_system, 9 links, 8 joints
Links:
- removed link base
- removed link gantry_x
- removed link gantry_y
- removed link link1
- removed link link2
- removed link link3
- removed link link4
- removed link link5
- removed link link6
- added link carriage, mass 645.33; collision mesh filename=package://shimizu_gantry_system/meshes/carriage.STL; visual mesh filename=package://shimizu_gantry_system/meshes/carriage.STL
- added link link_1, mass 39.488; collision mesh filename=package://shimizu_gantry_system/meshes/link_1.STL; visual mesh filename=package://shimizu_gantry_system/meshes/link_1.STL
- added link link_2, mass 26.224; collision mesh filename=package://shimizu_gantry_system/meshes/link_2.STL; visual mesh filename=package://shimizu_gantry_system/meshes/link_2.STL
- added link link_3, mass 41.069; collision mesh filename=package://shimizu_gantry_system/meshes/link_3.STL; visual mesh filename=package://shimizu_gantry_system/meshes/link_3.STL
- added link link_4, mass 2.0071; collision mesh filename=package://shimizu_gantry_system/meshes/link_4.STL; visual mesh filename=package://shimizu_gantry_system/meshes/link_4.STL
- added link link_5, mass 3.6409; collision mesh filename=package://shimizu_gantry_system/meshes/link_5.STL; visual mesh filename=package://shimizu_gantry_system/meshes/link_5.STL
- added link link_6, mass 0.22702; collision mesh filename=package://shimizu_gantry_system/meshes/link_6.STL; visual mesh filename=package://shimizu_gantry_system/meshes/link_6.STL
- added link structure, mass 12293; collision mesh filename=package://shimizu_gantry_system/meshes/structure.STL; visual mesh filename=package://shimizu_gantry_system/meshes/structure.STL
- added link x_rail, mass 740.03; collision mesh filename=package://shimizu_gantry_system/meshes/x_rail.STL; visual mesh filename=package://shimizu_gantry_system/meshes/x_rail.STL
Joints:
- removed joint joint1
- removed joint joint2
- removed joint joint3
- removed joint joint4
- removed joint joint5
- removed joint joint6
- removed joint x_to_y
- removed joint y_to_base
- added joint joint_1: type continuous, parent carriage, child link_1, origin xyz=0 0 0.2635 rpy=0 0 0.0062665, axis 0 0 1
- added joint joint_2: type continuous, parent link_1, child link_2, origin xyz=0.32 0.08996 0.1865 rpy=0 0 0, axis 0 1 0
- added joint joint_3: type continuous, parent link_2, child link_3, origin xyz=0 -0.00496 0.87 rpy=0 0 0, axis 0 1 0
- added joint joint_4: type continuous, parent link_3, child link_4, origin xyz=0.82052 -0.085 0.225 rpy=0 0 0, axis 1 0 0
- added joint joint_5: type continuous, parent link_4, child link_5, origin xyz=0.1945 -0.04579 0 rpy=0 0 0, axis 0 1 0
- added joint joint_6: type continuous, parent link_5, child link_6, origin xyz=0.175 0.0422 0 rpy=0 0 0, axis 1 0 0
- added joint joint_rail_carriage: type prismatic, parent x_rail, child carriage, origin xyz=2.0675 0.184 -1.1204 rpy=3.1416 0 0, axis -1 0 0, limit lower=0 upper=0 effort=0 velocity=0
- added joint joint_structure_rail: type prismatic, parent structure, child x_rail, origin xyz=1.0082 3.756 3.7013 rpy=0 0 0, axis 0 1 0, limit lower=0 upper=0 effort=0 velocity=0
