Commit message: [Hw] adding urdf_shimizu_gantry

File: urdf_shimizu_gantry/urdf/urdf_shimizu_gantry.urdf (robot description, URDF)
Before this commit: robot shimizu_gantry_system, 9 links, 8 joints
Links:
- link carriage: mass 645.33 -> 645.325992510266; geometry collision mesh filename=package://urdf_shimizu_gantry/meshes/carriage.STL; visual mesh filename=package://urdf_shimizu_gantry/meshes/carriage.STL
- link link_1: mass 39.488 -> 39.4879875307153; geometry collision mesh filename=package://urdf_shimizu_gantry/meshes/link_1.STL; visual mesh filename=package://urdf_shimizu_gantry/meshes/link_1.STL
- link link_2: mass 26.224 -> 26.2236990697048; geometry collision mesh filename=package://urdf_shimizu_gantry/meshes/link_2.STL; visual mesh filename=package://urdf_shimizu_gantry/meshes/link_2.STL
- link link_3: mass 41.069 -> 41.0689199450586; geometry collision mesh filename=package://urdf_shimizu_gantry/meshes/link_3.STL; visual mesh filename=package://urdf_shimizu_gantry/meshes/link_3.STL
- link link_4: mass 2.0071 -> 2.00706266186349; geometry collision mesh filename=package://urdf_shimizu_gantry/meshes/link_4.STL; visual mesh filename=package://urdf_shimizu_gantry/meshes/link_4.STL
- link link_5: mass 3.6409 -> 3.64087786116007; geometry collision mesh filename=package://urdf_shimizu_gantry/meshes/link_5.STL; visual mesh filename=package://urdf_shimizu_gantry/meshes/link_5.STL
- link link_6: mass 0.22702 -> 0.227022546438295; geometry collision mesh filename=package://urdf_shimizu_gantry/meshes/link_6.STL; visual mesh filename=package://urdf_shimizu_gantry/meshes/link_6.STL
- link structure: mass 12293 -> 12293.2154089237; geometry collision mesh filename=package://urdf_shimizu_gantry/meshes/structure.STL; visual mesh filename=package://urdf_shimizu_gantry/meshes/structure.STL
- link x_rail: mass 740.03 -> 740.030344861601; geometry collision mesh filename=package://urdf_shimizu_gantry/meshes/x_rail.STL; visual mesh filename=package://urdf_shimizu_gantry/meshes/x_rail.STL
Joints:
- joint joint_1: limit (none) -> lower=0 upper=6.28 effort=0 velocity=2.97
- joint joint_2: limit (none) -> lower=0 upper=4.28 effort=0 velocity=2.44
- joint joint_3: limit (none) -> lower=0 upper=6.28 effort=0 velocity=2.79
- joint joint_4: limit (none) -> lower=0 upper=12.57 effort=0 velocity=4.01
- joint joint_5: limit (none) -> lower=0 upper=4.36 effort=0 velocity=4.01
- joint joint_6: limit (none) -> lower=0 upper=12.57 effort=0 velocity=6.11
- joint joint_rail_carriage: limit lower=0 upper=0 effort=0 velocity=0 -> lower=0 upper=4.6411 effort=0 velocity=2; origin xyz=2.0675 0.184 -1.1204 rpy=3.1416 0 0 -> xyz=0.77533 0.184 -1.1204 rpy=3.1416 0 0
- joint joint_structure_rail: limit lower=0 upper=0 effort=0 velocity=0 -> lower=0 upper=6.1489 effort=0 velocity=2; origin xyz=1.0082 3.756 3.7013 rpy=0 0 0 -> xyz=1.0082 1.4226 3.7013 rpy=0 0 0

Commit message: [Hw] revise urdf file, x axis direction

File: urdf_shimizu_gantry/urdf/urdf_shimizu_gantry.urdf (robot description, URDF)
Before this commit: robot urdf_shimizu_gantry, 9 links, 8 joints
Joints:
- joint joint_rail_carriage: axis -1 0 0 -> 1 0 0
